File: BTS.brd (EAGLE design)
At the start: 115.6 x 84.5 mm, 55 parts, among them IC1 TPA3140D2PWP, IC2 BLK-MD-SPK-B, J1 SPKR_OUT, J2 RN52BoB_R, J3 RN52BoB_L, J6 HC-05, J7 PRT-10474, T3_2 TEENSY_3.1-3.2_DIL

Commit message: v1.0 for PCB fabrication
Parts:
- moved T3_2 1.91 mm to (99.7, 29.2)
Routing:
- net GPIO10: track 172.5 -> 169.2 mm
- net 3V3: track 225.8 -> 223.7 mm
- net STATE: track 181.3 -> 179.4 mm
- net HC_UART_RX: track 145.5 -> 143.6 mm
- net HC_UART_TX: track 138.8 -> 136.9 mm
- net GPIO5: track 152.2 -> 150.2 mm
- net SHUTDOWN: track 20.0 -> 18.1 mm
- net GPIO4: track 148.4 -> 146.5 mm
- net GPIO2: track 113.9 -> 112.0 mm
- net GPIO3: track 133.9 -> 132.1 mm
- net UART_RX: track 114.3 -> 112.8 mm
- net UART_TX: track 117.6 -> 116.5 mm
- net GPIO11: track 164.4 -> 163.6 mm
- net GPIO9: track 137.1 -> 136.3 mm
Other:
- board size 115.6 x 84.5 mm -> 113 x 84.5 mm
