File: Hardware/BTS_V2.brd (EAGLE design)
At the start: 113 x 79.4 mm, 63 parts, among them IC1 TPA3140D2PWP, IC2 BLK-MD-SPK-B, J1 SPKR_OUT, J2 RN52BoB_R, J3 RN52BoB_L, J4 TFT_CONNECTION, J6 HC-05, T3_2 TEENSY_3.1-3.2_DIL

Commit message: Board errors corrected
Parts:
- added C21: 1.0uF, SparkFun-Capacitors:0603
Connections:
- removed net LIMRATE: IC1.5, R5.2
- net GND: now also C21.2
- net GVDD: now also C21.1, IC1.5, R5.2
Routing:
- net GVDD: track 20.5 -> 79.4 mm, vias 2 -> 4
- net LIMRATE: track 40.4 -> 0.00 mm, vias 2 -> 0
Other:
- board text added: "C - 04/2018"
- board text removed: "C - 03/2018"
Changed lines of the file:
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@@
 <text x="6.985" y="5.715" size="1.778" layer="21">BTS</text>
 <text x="22.86" y="5.08" size="6.4516" layer="22" rot="MR0">REAR</text>
-<text x="109.855" y="5.08" size="6.4516" layer="22" rot="MR0">C - 03/2018</text>
+<text x="109.855" y="5.08" size="6.4516" layer="22" rot="MR0">C - 04/2018</text>
 <wire x1="4.445" y1="13.335" x2="4.445" y2="28.575" width="1.27" layer="22" style="longdash"/>
 <wire x1="4.445" y1="28.575" x2="26.67" y2="28.575" width="1.27" layer="22" style="longdash"/>
@@
 <text x="87.63" y="76.835" size="1.016" layer="21">VIN</text>
 <text x="87.63" y="70.485" size="1.016" layer="21">PVCC</text>
+<text x="57.785" y="22.225" size="1.778" layer="21" font="vector" rot="R270">1uF</text>
+<wire x1="59.69" y1="21.336" x2="59.69" y2="19.3548" width="0.1524" layer="21"/>
+<wire x1="59.69" y1="19.3294" x2="63.4746" y2="19.3294" width="0.1524" layer="21"/>
+<wire x1="63.4746" y1="19.3294" x2="63.4746" y2="21.336" width="0.1524" layer="21"/>
+<wire x1="63.4746" y1="21.336" x2="59.69" y2="21.336" width="0.1524" layer="21"/>
 </plain>
 <attributes>
@@
 <attribute name="TP_SIGNAL_NAME" value="" x="7.62" y="62.23" size="1.778" layer="27" display="off"/>
 </element>
+<element name="C21" library="SparkFun-Capacitors" library_urn="urn:adsk.eagle:library:510" package="0603" package3d_urn="urn:adsk.eagle:package:37414/1" value="1.0uF" x="61.595" y="20.32">
+<attribute name="PROD_ID" value="CAP-00868" x="61.595" y="20.32" size="1.778" layer="27" display="off"/>
+</element>
 </elements>
 <signals>
@@
 <vertex x="113.03" y="79.375"/>
 </polygon>
+<contactref element="C21" pad="2"/>
 </signal>
 <signal name="N$1">
@@
 <wire x1="60.745" y1="32.385" x2="60.745" y2="29.845" width="0.4064" layer="1"/>
 </signal>
-<signal name="GVDD">
-<contactref element="R2" pad="1"/>
-<contactref element="IC1" pad="9"/>
-<wire x1="60.745" y1="34.925" x2="59.055" y2="34.925" width="0.4064" layer="1"/>
-<via x="59.055" y="34.925" extent="1-16" drill="0.35"/>
-<wire x1="59.055" y1="34.925" x2="71.453" y2="34.925" width="0.4064" layer="16"/>
-<wire x1="71.453" y1="34.925" x2="72.2376" y2="35.8366" width="0.4064" layer="16"/>
-<via x="72.2376" y="35.8366" extent="1-16" drill="0.35"/>
-<wire x1="72.2404" y1="33.3177875" x2="72.2404" y2="32.5952125" width="0.4064" layer="1"/>
-<wire x1="72.2404" y1="32.5952125" x2="72.685" y2="32.3030125" width="0.4064" layer="1"/>
-<wire x1="72.685" y1="32.3030125" x2="72.685" y2="30.878" width="0.4064" layer="1"/>
-<wire x1="72.2376" y1="35.8366" x2="72.2376" y2="33.9245875" width="0.4064" layer="1"/>
-<wire x1="72.2376" y1="33.9245875" x2="72.2404" y2="33.3177875" width="0.4064" layer="1"/>
-</signal>
 <signal name="GAIN">
 <contactref element="IC1" pad="6"/>
@@
 <wire x1="71.12" y1="29.845" x2="71.755" y2="30.48" width="0.4064" layer="16"/>
 <wire x1="71.755" y1="30.48" x2="71.755" y2="32.385" width="0.4064" layer="16"/>
-</signal>
-<signal name="LIMRATE">
-<contactref element="IC1" pad="5"/>
-<contactref element="R5" pad="2"/>
-<wire x1="62.445" y1="24.765" x2="63.5" y2="24.765" width="0.4064" layer="1"/>
-<wire x1="63.5" y1="24.765" x2="66.3702" y2="21.8948" width="0.4064" layer="1"/>
-<wire x1="67.1576" y1="21.8948" x2="67.183" y2="21.9202" width="0.4064" layer="1"/>
-<via x="67.183" y="21.9202" extent="1-16" drill="0.35"/>
-<wire x1="67.183" y1="21.9202" x2="78.4352" y2="21.9202" width="0.4064" layer="16"/>
-<wire x1="78.4352" y1="21.9202" x2="80.645" y2="24.13" width="0.4064" layer="16"/>
-<wire x1="80.645" y1="24.13" x2="80.645" y2="32.385" width="0.4064" layer="16"/>
-<wire x1="77.47" y1="35.56" x2="74.93" y2="35.56" width="0.4064" layer="16"/>
-<via x="74.93" y="35.56" extent="1-16" drill="0.35"/>
-<wire x1="74.93" y1="35.56" x2="74.93" y2="33.655" width="0.4064" layer="1"/>
-<wire x1="66.3702" y1="21.8948" x2="67.1576" y2="21.8948" width="0.4064" layer="1"/>
-<wire x1="80.645" y1="32.385" x2="77.47" y2="35.56" width="0.4064" layer="16"/>
-<wire x1="75.285" y1="30.878" x2="75.2856" y2="30.8786" width="0.4064" layer="1"/>
-<wire x1="75.2856" y1="30.8786" x2="75.2856" y2="33.2994" width="0.4064" layer="1"/>
-<wire x1="75.2856" y1="33.2994" x2="74.93" y2="33.655" width="0.4064" layer="1"/>
 </signal>
 <signal name="RINN">
@@
 <wire x1="97.79" y1="18.415" x2="97.79" y2="19.685" width="0.4064" layer="16"/>
 </signal>
+<signal name="GVDD">
+<contactref element="IC1" pad="5"/>
+<contactref element="R5" pad="2"/>
+<contactref element="R2" pad="1"/>
+<contactref element="IC1" pad="9"/>
+<wire x1="62.445" y1="24.765" x2="63.5" y2="24.765" width="0.4064" layer="1"/>
+<wire x1="64.135" y1="24.13" x2="63.5" y2="24.765" width="0.4064" layer="1"/>
+<wire x1="64.135" y1="21.9202" x2="78.4352" y2="21.9202" width="0.4064" layer="16"/>
+<wire x1="78.4352" y1="21.9202" x2="80.645" y2="24.13" width="0.4064" layer="16"/>
+<wire x1="80.645" y1="24.13" x2="80.645" y2="32.385" width="0.4064" layer="16"/>
+<wire x1="77.47" y1="35.56" x2="74.93" y2="35.56" width="0.4064" layer="16"/>
+<via x="74.93" y="35.56" extent="1-16" drill="0.35"/>
+<wire x1="74.93" y1="35.56" x2="74.93" y2="33.655" width="0.4064" layer="1"/>
+<wire x1="80.645" y1="32.385" x2="77.47" y2="35.56" width="0.4064" layer="16"/>
+<wire x1="75.285" y1="30.878" x2="75.2856" y2="30.8786" width="0.4064" layer="1"/>
+<wire x1="75.2856" y1="30.8786" x2="75.2856" y2="33.2994" width="0.4064" layer="1"/>
+<wire x1="75.2856" y1="33.2994" x2="74.93" y2="33.655" width="0.4064" layer="1"/>
+<wire x1="60.745" y1="34.925" x2="59.055" y2="34.925" width="0.4064" layer="1"/>
+<via x="59.055" y="34.925" extent="1-16" drill="0.35"/>
+<wire x1="59.055" y1="34.925" x2="71.453" y2="34.925" width="0.4064" layer="16"/>
+<wire x1="71.453" y1="34.925" x2="72.2376" y2="35.8366" width="0.4064" layer="16"/>
+<via x="72.2376" y="35.8366" extent="1-16" drill="0.35"/>
+<wire x1="72.2404" y1="33.3177875" x2="72.2404" y2="32.5952125" width="0.4064" layer="1"/>
+<wire x1="72.2404" y1="32.5952125" x2="72.685" y2="32.3030125" width="0.4064" layer="1"/>
+<wire x1="72.685" y1="32.3030125" x2="72.685" y2="30.878" width="0.4064" layer="1"/>
+<wire x1="72.2376" y1="35.8366" x2="72.2376" y2="33.9245875" width="0.4064" layer="1"/>
+<wire x1="72.2376" y1="33.9245875" x2="72.2404" y2="33.3177875" width="0.4064" layer="1"/>
+<wire x1="59.055" y1="23.495" x2="59.055" y2="34.925" width="0.4064" layer="16"/>
+<wire x1="59.055" y1="23.495" x2="60.6298" y2="21.9202" width="0.4064" layer="16"/>
+<via x="64.135" y="21.9202" extent="1-16" drill="0.35"/>
+<wire x1="60.6298" y1="21.9202" x2="64.135" y2="21.9202" width="0.4064" layer="16"/>
+<wire x1="64.135" y1="21.9202" x2="64.135" y2="24.13" width="0.4064" layer="1"/>
+<contactref element="C21" pad="1"/>
+<wire x1="60.745" y1="20.32" x2="60.6298" y2="21.9202" width="0" layer="19" extent="1-16"/>
+</signal>
 </signals>

Commit message: Still working on figuring out an error w/ the board
Changed lines of the file:
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@@
 <wire x1="33.64" y1="29.03" x2="47.64" y2="29.03" width="0.4064" layer="1"/>
 <via x="71.755" y="28.956" extent="1-16" drill="0.55"/>
-<via x="70.1294" y="27.94" extent="1-16" drill="0.55"/>
+<via x="70.358" y="27.94" extent="1-16" drill="0.55"/>
 <via x="71.755" y="26.924" extent="1-16" drill="0.55"/>
 <via x="73.025" y="26.924" extent="1-16" drill="0.55"/>
