File: Hardware/BTS_V2.sch (EAGLE design)
At the start: 57 parts, among them IC1 TPA3140D2PWP, IC2 BLK-MD-SPK-B, J1 SPKR_OUT, J2 RN52BoB_R, J3 RN52BoB_L, J6 HC-05, J7 PRT-10474, T3_2 TEENSY_3.1-3.2_DIL

Commit message: Created new XT-60 connector
Parts:
- added U$1: HK_XT-60, myLib:HK_XT-60
Connections:
- net GND: now also U$1.NEG
- net VIN: now also U$1.POS
Changed lines of the file:
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@@
 <part name="R16" library="resistor" library_urn="urn:adsk.eagle:library:348" deviceset="R-US_" device="R0603" package3d_urn="urn:adsk.eagle:package:26057/1" value="100R"/>
 <part name="GND12" library="supply1" library_urn="urn:adsk.eagle:library:371" deviceset="GND" device=""/>
+<part name="U$1" library="myLib" deviceset="HK_XT-60" device=""/>
 </parts>
 <sheets>
@@
 <instance part="R16" gate="G$1" x="132.08" y="235.204" rot="R90"/>
 <instance part="GND12" gate="1" x="172.72" y="237.236"/>
+<instance part="U$1" gate="G$1" x="195.58" y="198.12"/>
 </instances>
 <busses>
@@
 <wire x1="218.44" y1="187.96" x2="220.98" y2="187.96" width="0.1524" layer="91"/>
 <wire x1="220.98" y1="187.96" x2="220.98" y2="186.436" width="0.1524" layer="91"/>
+<pinref part="U$1" gate="G$1" pin="NEG"/>
+<wire x1="203.2" y1="203.2" x2="226.06" y2="203.2" width="0.1524" layer="91"/>
+<wire x1="226.06" y1="203.2" x2="226.06" y2="187.96" width="0.1524" layer="91"/>
+<wire x1="226.06" y1="187.96" x2="220.98" y2="187.96" width="0.1524" layer="91"/>
+<junction x="220.98" y="187.96"/>
 </segment>
 <segment>
@@
 <pinref part="C7" gate="G$1" pin="1"/>
 <wire x1="261.62" y1="187.96" x2="261.62" y2="190.5" width="0.1524" layer="91"/>
-<wire x1="218.44" y1="190.5" x2="231.14" y2="190.5" width="0.1524" layer="91"/>
+<wire x1="218.44" y1="190.5" x2="220.98" y2="190.5" width="0.1524" layer="91"/>
 <label x="220.98" y="190.5" size="1.778" layer="95"/>
+<wire x1="220.98" y1="190.5" x2="231.14" y2="190.5" width="0.1524" layer="91"/>
 <wire x1="231.14" y1="190.5" x2="261.62" y2="190.5" width="0.1524" layer="91"/>
 <wire x1="276.86" y1="190.5" x2="261.62" y2="190.5" width="0.1524" layer="91"/>
@@
 <wire x1="276.86" y1="205.74" x2="276.86" y2="190.5" width="0.1524" layer="91"/>
 <pinref part="J7" gate="G$1" pin="POS"/>
-</segment>
-</net>
+<wire x1="220.98" y1="190.5" x2="220.98" y2="198.12" width="0.1524" layer="91"/>
+<junction x="220.98" y="190.5"/>
+<pinref part="U$1" gate="G$1" pin="POS"/>
+<wire x1="220.98" y1="198.12" x2="203.2" y2="198.12" width="0.1524" layer="91"/>
+</segment>
+</net>

Commit message: added PA test code & modified V2 board files
Parts:
- removed J7: PRT-10474, PRT-10474:PRT-10474
- added TP1, TP2, TP3, TP4, TP5, TP6: TPSPAD1-17, testpad:TPSPAD1-17
- J4: value (none) -> TFT_CONNECTION
Connections:
- net 3V3: now also TP2.PP
- net GND: now also TP6.PP; no longer J7.GND
- net PVCC: now also TP1.PP
- net SPKR_L+: now also TP4.PP
- net SPKR_L-: now also TP5.PP
- net VIN: now also TP3.PP; no longer J7.POS
Changed lines of the file:
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@@
 <part name="PAD1" library="wirepad" library_urn="urn:adsk.eagle:library:412" deviceset="SMD2" device="" package3d_urn="urn:adsk.eagle:package:30839/1" value="?"/>
 <part name="PAD2" library="wirepad" library_urn="urn:adsk.eagle:library:412" deviceset="SMD2" device="" package3d_urn="urn:adsk.eagle:package:30839/1" value="?"/>
-<part name="J7" library="PRT-10474" deviceset="PRT-10474" device=""/>
 <part name="GND11" library="supply1" library_urn="urn:adsk.eagle:library:371" deviceset="GND" device=""/>
 <part name="T3_2" library="Teensy_3_and_LC_Series_Boards_v1.4" deviceset="TEENSY_3.1-3.2_DIL" device=""/>
@@
 <attribute name="RESISTANCE" value="33K"/>
 </part>
-<part name="J4" library="SparkFun-Connectors" library_urn="urn:adsk.eagle:library:513" deviceset="CONN_14" device="" package3d_urn="urn:adsk.eagle:package:38183/1"/>
+<part name="J4" library="SparkFun-Connectors" library_urn="urn:adsk.eagle:library:513" deviceset="CONN_14" device="" package3d_urn="urn:adsk.eagle:package:38183/1" value="TFT_CONNECTION"/>
 <part name="R16" library="resistor" library_urn="urn:adsk.eagle:library:348" deviceset="R-US_" device="R0603" package3d_urn="urn:adsk.eagle:package:26057/1" value="100R"/>
 <part name="GND12" library="supply1" library_urn="urn:adsk.eagle:library:371" deviceset="GND" device=""/>
 <part name="U$1" library="myLib" deviceset="HK_XT-60" device=""/>
+<part name="TP1" library="testpad" library_urn="urn:adsk.eagle:library:385" deviceset="TPS" device="PAD1-17" package3d_urn="urn:adsk.eagle:package:27949/1"/>
+<part name="TP2" library="testpad" library_urn="urn:adsk.eagle:library:385" deviceset="TPS" device="PAD1-17" package3d_urn="urn:adsk.eagle:package:27949/1"/>
+<part name="TP3" library="testpad" library_urn="urn:adsk.eagle:library:385" deviceset="TPS" device="PAD1-17" package3d_urn="urn:adsk.eagle:package:27949/1"/>
+<part name="TP4" library="testpad" library_urn="urn:adsk.eagle:library:385" deviceset="TPS" device="PAD1-17" package3d_urn="urn:adsk.eagle:package:27949/1"/>
+<part name="TP5" library="testpad" library_urn="urn:adsk.eagle:library:385" deviceset="TPS" device="PAD1-17" package3d_urn="urn:adsk.eagle:package:27949/1"/>
+<part name="TP6" library="testpad" library_urn="urn:adsk.eagle:library:385" deviceset="TPS" device="PAD1-17" package3d_urn="urn:adsk.eagle:package:27949/1"/>
+<part name="GND13" library="supply1" library_urn="urn:adsk.eagle:library:371" deviceset="GND" device=""/>
 </parts>
 <sheets>
@@
 <instance part="PAD1" gate="1" x="63.5" y="187.96" rot="R180"/>
 <instance part="PAD2" gate="1" x="63.5" y="185.42" rot="R180"/>
-<instance part="J7" gate="G$1" x="218.44" y="187.96" rot="R180"/>
-<instance part="GND11" gate="1" x="220.98" y="183.896"/>
+<instance part="GND11" gate="1" x="231.648" y="193.04"/>
 <instance part="T3_2" gate="G$1" x="101.6" y="152.4"/>
 <instance part="R15" gate="G$1" x="208.28" y="88.9" rot="R270"/>
@@
 <instance part="R16" gate="G$1" x="132.08" y="235.204" rot="R90"/>
 <instance part="GND12" gate="1" x="172.72" y="237.236"/>
-<instance part="U$1" gate="G$1" x="195.58" y="198.12"/>
+<instance part="U$1" gate="G$1" x="205.74" y="190.5"/>
+<instance part="TP1" gate="G$1" x="325.12" y="228.6"/>
+<instance part="TP2" gate="G$1" x="375.92" y="177.8" rot="R270"/>
+<instance part="TP3" gate="G$1" x="238.76" y="200.66"/>
+<instance part="TP4" gate="G$1" x="162.56" y="91.44"/>
+<instance part="TP5" gate="G$1" x="167.64" y="91.44"/>
+<instance part="TP6" gate="G$1" x="213.36" y="238.76"/>
+<instance part="GND13" gate="1" x="213.36" y="231.14"/>
 </instances>
 <busses>
@@
 </segment>
 <segment>
-<pinref part="J7" gate="G$1" pin="GND"/>
 <pinref part="GND11" gate="1" pin="GND"/>
-<wire x1="218.44" y1="187.96" x2="220.98" y2="187.96" width="0.1524" layer="91"/>
-<wire x1="220.98" y1="187.96" x2="220.98" y2="186.436" width="0.1524" layer="91"/>
+<wire x1="213.36" y1="195.58" x2="231.648" y2="195.58" width="0.1524" layer="91"/>
 <pinref part="U$1" gate="G$1" pin="NEG"/>
-<wire x1="203.2" y1="203.2" x2="226.06" y2="203.2" width="0.1524" layer="91"/>
-<wire x1="226.06" y1="203.2" x2="226.06" y2="187.96" width="0.1524" layer="91"/>
-<wire x1="226.06" y1="187.96" x2="220.98" y2="187.96" width="0.1524" layer="91"/>
-<junction x="220.98" y="187.96"/>
 </segment>
 <segment>
@@
 <wire x1="149.86" y1="241.3" x2="172.72" y2="241.3" width="0.1524" layer="91"/>
 <wire x1="172.72" y1="241.3" x2="172.72" y2="239.776" width="0.1524" layer="91"/>
+</segment>
+<segment>
+<pinref part="GND13" gate="1" pin="GND"/>
+<pinref part="TP6" gate="G$1" pin="PP"/>
+<wire x1="213.36" y1="233.68" x2="213.36" y2="236.22" width="0.1524" layer="91"/>
 </segment>
 </net>
@@
 <wire x1="309.88" y1="213.36" x2="309.88" y2="218.44" width="0.1524" layer="91"/>
 <junction x="309.88" y="213.36"/>
-<wire x1="330.708" y1="218.44" x2="309.88" y2="218.44" width="0.1524" layer="91"/>
+<wire x1="330.708" y1="218.44" x2="325.12" y2="218.44" width="0.1524" layer="91"/>
 <pinref part="C10" gate="G$1" pin="1"/>
+<wire x1="325.12" y1="218.44" x2="309.88" y2="218.44" width="0.1524" layer="91"/>
 <wire x1="330.708" y1="217.17" x2="330.708" y2="218.44" width="0.1524" layer="91"/>
 <wire x1="330.708" y1="218.44" x2="342.138" y2="218.44" width="0.1524" layer="91"/>
@@
 <label x="362.458" y="218.44" size="1.778" layer="95"/>
 <junction x="330.708" y="218.44"/>
+<pinref part="TP1" gate="G$1" pin="PP"/>
+<wire x1="325.12" y1="226.06" x2="325.12" y2="218.44" width="0.1524" layer="91"/>
+<junction x="325.12" y="218.44"/>
 </segment>
 </net>
@@
 <pinref part="J2" gate="G$1" pin="20"/>
 <label x="139.7" y="86.36" size="1.778" layer="95"/>
-<wire x1="137.16" y1="86.36" x2="185.42" y2="86.36" width="0.1524" layer="91"/>
+<wire x1="137.16" y1="86.36" x2="162.56" y2="86.36" width="0.1524" layer="91"/>
+<wire x1="162.56" y1="86.36" x2="185.42" y2="86.36" width="0.1524" layer="91"/>
 <wire x1="185.42" y1="86.36" x2="185.42" y2="78.74" width="0.1524" layer="91"/>
 <pinref part="C1" gate="G$1" pin="1"/>
@@
 <wire x1="137.16" y1="86.36" x2="63.5" y2="86.36" width="0.1524" layer="91"/>
 <junction x="137.16" y="86.36"/>
+<pinref part="TP4" gate="G$1" pin="PP"/>
+<wire x1="162.56" y1="86.36" x2="162.56" y2="88.9" width="0.1524" layer="91"/>
+<junction x="162.56" y="86.36"/>
 </segment>
 </net>
@@
 <pinref part="J2" gate="G$1" pin="19"/>
 <label x="139.7" y="83.82" size="1.778" layer="95"/>
-<wire x1="137.16" y1="83.82" x2="180.34" y2="83.82" width="0.1524" layer="91"/>
+<wire x1="137.16" y1="83.82" x2="167.64" y2="83.82" width="0.1524" layer="91"/>
 <pinref part="C2" gate="G$1" pin="1"/>
+<wire x1="167.64" y1="83.82" x2="180.34" y2="83.82" width="0.1524" layer="91"/>
 <wire x1="180.34" y1="83.82" x2="180.34" y2="76.2" width="0.1524" layer="91"/>
 <wire x1="180.34" y1="76.2" x2="190.5" y2="76.2" width="0.1524" layer="91"/>
@@
 <wire x1="137.16" y1="83.82" x2="111.76" y2="83.82" width="0.1524" layer="91"/>
 <junction x="137.16" y="83.82"/>
+<pinref part="TP5" gate="G$1" pin="PP"/>
+<wire x1="167.64" y1="83.82" x2="167.64" y2="88.9" width="0.1524" layer="91"/>
+<junction x="167.64" y="83.82"/>
 </segment>
 </net>
@@
 <pinref part="C7" gate="G$1" pin="1"/>
 <wire x1="261.62" y1="187.96" x2="261.62" y2="190.5" width="0.1524" layer="91"/>
-<wire x1="218.44" y1="190.5" x2="220.98" y2="190.5" width="0.1524" layer="91"/>
-<label x="220.98" y="190.5" size="1.778" layer="95"/>
-<wire x1="220.98" y1="190.5" x2="231.14" y2="190.5" width="0.1524" layer="91"/>
-<wire x1="231.14" y1="190.5" x2="261.62" y2="190.5" width="0.1524" layer="91"/>
+<label x="215.9" y="190.5" size="1.778" layer="95"/>
+<wire x1="213.36" y1="190.5" x2="231.14" y2="190.5" width="0.1524" layer="91"/>
+<wire x1="231.14" y1="190.5" x2="238.76" y2="190.5" width="0.1524" layer="91"/>
+<wire x1="238.76" y1="190.5" x2="261.62" y2="190.5" width="0.1524" layer="91"/>
 <wire x1="276.86" y1="190.5" x2="261.62" y2="190.5" width="0.1524" layer="91"/>
 <junction x="276.86" y="190.5"/>
@@
 <wire x1="281.94" y1="205.74" x2="276.86" y2="205.74" width="0.1524" layer="91"/>
 <wire x1="276.86" y1="205.74" x2="276.86" y2="190.5" width="0.1524" layer="91"/>
-<pinref part="J7" gate="G$1" pin="POS"/>
-<wire x1="220.98" y1="190.5" x2="220.98" y2="198.12" width="0.1524" layer="91"/>
-<junction x="220.98" y="190.5"/>
 <pinref part="U$1" gate="G$1" pin="POS"/>
-<wire x1="220.98" y1="198.12" x2="203.2" y2="198.12" width="0.1524" layer="91"/>
+<pinref part="TP3" gate="G$1" pin="PP"/>
+<wire x1="238.76" y1="198.12" x2="238.76" y2="190.5" width="0.1524" layer="91"/>
+<junction x="238.76" y="190.5"/>
 </segment>
 </net>
@@
 <pinref part="C8" gate="G$1" pin="1"/>
 <wire x1="353.06" y1="175.26" x2="353.06" y2="177.8" width="0.1524" layer="91"/>
-<wire x1="353.06" y1="177.8" x2="365.76" y2="177.8" width="0.1524" layer="91"/>
+<wire x1="353.06" y1="177.8" x2="373.38" y2="177.8" width="0.1524" layer="91"/>
 <pinref part="L5" gate="G$1" pin="2"/>
 <wire x1="350.52" y1="177.8" x2="353.06" y2="177.8" width="0.1524" layer="91"/>
 <junction x="353.06" y="177.8"/>
 <label x="365.76" y="177.8" size="1.778" layer="95"/>
-</segment>
-<segment>
+<pinref part="TP2" gate="G$1" pin="PP"/>
+</segment>
+<segment>

Commit message: Board errors corrected
Parts:
- added C21: 1.0uF, SparkFun-Capacitors:1.0UF-0603-16V-10%
Connections:
- removed net LIMRATE: IC1.LIMRATE, R5.2
- net GND: now also C21.2
- net GVDD: now also C21.1, IC1.LIMRATE, R5.2
Changed lines of the file:
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@@
 <part name="TP6" library="testpad" library_urn="urn:adsk.eagle:library:385" deviceset="TPS" device="PAD1-17" package3d_urn="urn:adsk.eagle:package:27949/1"/>
 <part name="GND13" library="supply1" library_urn="urn:adsk.eagle:library:371" deviceset="GND" device=""/>
+<part name="C21" library="SparkFun-Capacitors" library_urn="urn:adsk.eagle:library:510" deviceset="1.0UF" device="-0603-16V-10%" package3d_urn="urn:adsk.eagle:package:37414/1" value="1.0uF"/>
 </parts>
 <sheets>
@@
 <instance part="R5" gate="G$1" x="194.31" y="66.04"/>
 <instance part="R6" gate="G$1" x="181.61" y="66.04"/>
-<instance part="GND1" gate="1" x="165.1" y="58.42"/>
+<instance part="GND1" gate="1" x="165.1" y="56.388"/>
 <instance part="C1" gate="G$1" x="204.47" y="78.74" rot="R90"/>
 <instance part="C2" gate="G$1" x="195.58" y="76.2" rot="R90"/>
@@
 <instance part="TP6" gate="G$1" x="213.36" y="238.76"/>
 <instance part="GND13" gate="1" x="213.36" y="231.14"/>
+<instance part="C21" gate="G$1" x="168.91" y="60.96" rot="R270"/>
 </instances>
 <busses>
@@
 <pinref part="GND1" gate="1" pin="GND"/>
 <pinref part="R4" gate="G$1" pin="2"/>
+<wire x1="165.1" y1="58.928" x2="165.1" y2="60.96" width="0.1524" layer="91"/>
 <wire x1="165.1" y1="60.96" x2="165.1" y2="63.5" width="0.1524" layer="91"/>
 <wire x1="165.1" y1="63.5" x2="170.18" y2="63.5" width="0.1524" layer="91"/>
@@
 <wire x1="68.58" y1="66.04" x2="83.82" y2="66.04" width="0.1524" layer="91"/>
 <junction x="83.82" y="66.04"/>
+<pinref part="C21" gate="G$1" pin="2"/>
+<wire x1="166.37" y1="60.96" x2="165.1" y2="60.96" width="0.1524" layer="91"/>
+<junction x="165.1" y="60.96"/>
 </segment>
 <segment>
@@
 </segment>
 </net>
-<net name="GVDD" class="0">
-<segment>
-<pinref part="R2" gate="G$1" pin="1"/>
-<pinref part="IC1" gate="G$1" pin="GVDD"/>
-<wire x1="205.74" y1="63.5" x2="210.82" y2="63.5" width="0.1524" layer="91"/>
-</segment>
-</net>
 <net name="GAIN" class="0">
 <segment>
@@
 <wire x1="194.31" y1="63.5" x2="195.58" y2="63.5" width="0.1524" layer="91"/>
 <wire x1="210.82" y1="68.58" x2="208.28" y2="68.58" width="0.1524" layer="91"/>
-<wire x1="208.28" y1="68.58" x2="201.93" y2="68.58" width="0.1524" layer="91"/>
-<wire x1="194.31" y1="71.12" x2="194.31" y2="63.5" width="0.1524" layer="91"/>
+<wire x1="194.31" y1="68.58" x2="194.31" y2="63.5" width="0.1524" layer="91"/>
 <junction x="194.31" y="63.5"/>
-<wire x1="201.93" y1="68.58" x2="201.93" y2="71.12" width="0.1524" layer="91"/>
-<wire x1="201.93" y1="71.12" x2="194.31" y2="71.12" width="0.1524" layer="91"/>
+<wire x1="208.28" y1="68.58" x2="194.31" y2="68.58" width="0.1524" layer="91"/>
 <wire x1="208.28" y1="71.12" x2="208.28" y2="68.58" width="0.1524" layer="91"/>
 <junction x="208.28" y="68.58"/>
@@
 <pinref part="IC1" gate="G$1" pin="LIMTHRES"/>
 <wire x1="210.82" y1="66.04" x2="205.74" y2="66.04" width="0.1524" layer="91"/>
-<wire x1="205.74" y1="66.04" x2="205.74" y2="72.39" width="0.1524" layer="91"/>
+<wire x1="205.74" y1="66.04" x2="205.74" y2="71.12" width="0.1524" layer="91"/>
 <pinref part="R6" gate="G$1" pin="2"/>
 <pinref part="R5" gate="G$1" pin="1"/>
 <wire x1="186.69" y1="66.04" x2="187.96" y2="66.04" width="0.1524" layer="91"/>
 <wire x1="187.96" y1="66.04" x2="189.23" y2="66.04" width="0.1524" layer="91"/>
-<wire x1="187.96" y1="72.39" x2="187.96" y2="66.04" width="0.1524" layer="91"/>
+<wire x1="187.96" y1="71.12" x2="187.96" y2="66.04" width="0.1524" layer="91"/>
 <junction x="187.96" y="66.04"/>
-<wire x1="205.74" y1="72.39" x2="187.96" y2="72.39" width="0.1524" layer="91"/>
-</segment>
-</net>
-<net name="LIMRATE" class="0">
-<segment>
-<pinref part="IC1" gate="G$1" pin="LIMRATE"/>
-<wire x1="210.82" y1="73.66" x2="204.47" y2="73.66" width="0.1524" layer="91"/>
-<wire x1="204.47" y1="73.66" x2="204.47" y2="66.04" width="0.1524" layer="91"/>
-<pinref part="R5" gate="G$1" pin="2"/>
-<wire x1="204.47" y1="66.04" x2="199.39" y2="66.04" width="0.1524" layer="91"/>
+<wire x1="205.74" y1="71.12" x2="187.96" y2="71.12" width="0.1524" layer="91"/>
 </segment>
 </net>
@@
 </segment>
 </net>
+<net name="GVDD" class="0">
+<segment>
+<pinref part="IC1" gate="G$1" pin="LIMRATE"/>
+<wire x1="210.82" y1="73.66" x2="204.47" y2="73.66" width="0.1524" layer="91"/>
+<wire x1="204.47" y1="73.66" x2="204.47" y2="66.04" width="0.1524" layer="91"/>
+<pinref part="R5" gate="G$1" pin="2"/>
+<wire x1="204.47" y1="66.04" x2="199.39" y2="66.04" width="0.1524" layer="91"/>
+<wire x1="204.47" y1="66.04" x2="204.47" y2="64.77" width="0.1524" layer="91"/>
+<wire x1="204.47" y1="64.77" x2="208.28" y2="64.77" width="0.1524" layer="91"/>
+<pinref part="R2" gate="G$1" pin="1"/>
+<pinref part="IC1" gate="G$1" pin="GVDD"/>
+<wire x1="205.74" y1="63.5" x2="208.28" y2="63.5" width="0.1524" layer="91"/>
+<wire x1="208.28" y1="63.5" x2="210.82" y2="63.5" width="0.1524" layer="91"/>
+<wire x1="208.28" y1="64.77" x2="208.28" y2="63.5" width="0.1524" layer="91"/>
+<junction x="208.28" y="63.5"/>
+<pinref part="C21" gate="G$1" pin="1"/>
+<wire x1="173.99" y1="60.96" x2="208.28" y2="60.96" width="0.1524" layer="91"/>
+<wire x1="208.28" y1="60.96" x2="208.28" y2="63.5" width="0.1524" layer="91"/>
+</segment>
+</net>

Commit message: still tracking down issue
Parts:
- added TP7, TP8: TPSPAD1-17, testpad:TPSPAD1-17
Connections:
- net SPKR_R+: now also TP7.PP
- net SPKR_R-: now also TP8.PP
Other:
- moved on the sheet: C1, C13, C14, C15, C16, C17, C18, C19, C2, C20, C21, C3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
